File: pcb/pm_25.sch (KiCad schematic (older format))
At the start: 7 parts, among them J1 USB_B_Micro, U1 LD1117S33TR_TO220, U2 SI7021, U3 ESP-01v090, U4 Plantower-PM2.5

Commit message: make the PCB the same size as the plantower sensor
Parts:
- C2: footprint Capacitor_THT:CP_Radial_D5.0mm_P2.00mm -> Capacitor_THT:CP_Radial_D4.0mm_P2.00mm
Changed lines of the file:
@@
 F 0 "C2" H 5665 3846 50  0000 L CNN
 F 1 "10uF" H 5665 3755 50  0000 L CNN
-F 2 "Capacitor_THT:CP_Radial_D5.0mm_P2.00mm" H 5550 3800 50  0001 C CNN
+F 2 "Capacitor_THT:CP_Radial_D4.0mm_P2.00mm" H 5550 3800 50  0001 C CNN
 F 3 "~" H 5550 3800 50  0001 C CNN
 	1    5550 3800

Commit message: updating pcb
Parts:
- removed J1: USB_B_Micro, Connector_USB:USB_Mini-B_Lumberg_2486_01_Horizontal, symbol Connector:USB_B_Micro
- removed U1: LD1117S33TR_TO220, Package_TO_SOT_THT:TO-220-3_Horizontal_TabDown, symbol Regulator_Linear:LM1117-3.3
- removed U2: SI7021, pm_25:SI7021Breakout, symbol pm_25:SI7021
- removed U3: ESP-01v090, ESP8266:ESP-01, symbol ESP8266:ESP-01v090
- added C3: 47nf, Capacitor_THT:C_Disc_D4.7mm_W2.5mm_P5.00mm, symbol Device:C
- added H1, H2, H3, H4: MountingHole, MountingHole:MountingHole_2.5mm_Pad_Via, symbol Mechanical:MountingHole
- added J1: USB_C_Receptacle_USB2.0, Connector_USB:USB_C_Receptacle_GCT_USB4085, symbol Connector:USB_C_Receptacle_USB2.0
- added J2: header, Connector_PinSocket_2.54mm:PinSocket_1x04_P2.54mm_Vertical, symbol Connector_Generic:Conn_01x04
- added J3, J4: Qwiic, Connector_JST:JST_SH_BM04B-SRSS-TB_1x04-1MP_P1.00mm_Vertical, symbol Connector_Generic:Conn_01x04
- added R1, R2: 10k, Resistor_THT:R_Axial_DIN0207_L6.3mm_D2.5mm_P7.62mm_Horizontal, symbol Device:R
- added U1: MCP1700-3302E_TO92, Package_TO_SOT_THT:TO-92_Inline, symbol Regulator_Linear:MCP1700-3302E_TO92
- added U2: MCP2221AxP, Package_DIP:DIP-14_W7.62mm, symbol Interface_USB:MCP2221AxP
- added U3: ESP-12F, ESP8266:ESP-12E_SMD, symbol ESP8266:ESP-12F
- U4: footprint PMSX003-Breakout:0532610871 -> Connector_Molex:Molex_PicoBlade_53261-0871_1x08-1MP_P1.25mm_Horizontal
Connections:
- net labels added: D+, D-, FLASH, RST, SCL, SDA
- wire segments 35 -> 45
- no-connect marks 0 -> 17
Other:
- moved on the sheet: C1, C2, U4

Commit message: I guess Kicad wanted to change some stuff
Parts:
- U3: symbol ESP8266:ESP-12F -> pm_25-rescue:ESP-12F-ESP8266
Changed lines of the file:
@@
 	7250 3100 7250 3150
 $Comp
-L ESP8266:ESP-12F U3
+L pm_25-rescue:ESP-12F-ESP8266 U3
 U 1 1 600365AB
 P 8950 4200
@@
 	1    3350 5200
 	1    0    0    -1
-$EndComp
-$Comp
-L Connector_Generic:Conn_01x04 J3
-U 1 1 600889C9
-P 5300 6100
-F 0 "J3" V 5264 5812 50  0000 R CNN
-F 1 "Qwiic" V 5173 5812 50  0000 R CNN
-F 2 "Connector_JST:JST_SH_BM04B-SRSS-TB_1x04-1MP_P1.00mm_Vertical" H 5300 6100 50  0001 C CNN
-F 3 "~" H 5300 6100 50  0001 C CNN
-	1    5300 6100
-	0    -1   -1   0
 $EndComp
 $Comp
@@
 	6800 4600 6250 4600
 $Comp
+L power:GND #PWR0120
+U 1 1 600F9C99
+P 5100 6950
+F 0 "#PWR0120" H 5100 6700 50  0001 C CNN
+F 1 "GND" H 5105 6777 50  0000 C CNN
+F 2 "" H 5100 6950 50  0001 C CNN
+F 3 "" H 5100 6950 50  0001 C CNN
+	1    5100 6950
+	1    0    0    -1
+$EndComp
+Text Label 5450 6950 3    50   ~ 0
+SDA
+Text Label 5550 6950 3    50   ~ 0
+SCL
+Wire Wire Line
+	5250 6950 5100 6950
+$Comp
+L Connector_Generic:Conn_01x04 J3
+U 1 1 600889C9
+P 5300 6100
+F 0 "J3" V 5264 5812 50  0000 R CNN
+F 1 "Qwiic" V 5173 5812 50  0000 R CNN
+F 2 "Connector_JST:JST_SH_BM04B-SRSS-TB_1x04-1MP_P1.00mm_Vertical" H 5300 6100 50  0001 C CNN
+F 3 "~" H 5300 6100 50  0001 C CNN
+	1    5300 6100
+	0    -1   -1   0
+$EndComp
+$Comp
+L power:+3.3V #PWR0121
+U 1 1 600F9C9F
+P 5350 6950
+F 0 "#PWR0121" H 5350 6800 50  0001 C CNN
+F 1 "+3.3V" H 5365 7123 50  0000 C CNN
+F 2 "" H 5350 6950 50  0001 C CNN
+F 3 "" H 5350 6950 50  0001 C CNN
+	1    5350 6950
+	-1   0    0    1
+$EndComp
+$Comp
 L Connector_Generic:Conn_01x04 J4
 U 1 1 600F9C93
@@
 	0    -1   -1   0
 $EndComp
-$Comp
-L power:GND #PWR0120
-U 1 1 600F9C99
-P 5100 6950
-F 0 "#PWR0120" H 5100 6700 50  0001 C CNN
-F 1 "GND" H 5105 6777 50  0000 C CNN
-F 2 "" H 5100 6950 50  0001 C CNN
-F 3 "" H 5100 6950 50  0001 C CNN
-	1    5100 6950
-	1    0    0    -1
-$EndComp
-$Comp
-L power:+3.3V #PWR0121
-U 1 1 600F9C9F
-P 5350 6950
-F 0 "#PWR0121" H 5350 6800 50  0001 C CNN
-F 1 "+3.3V" H 5365 7123 50  0000 C CNN
-F 2 "" H 5350 6950 50  0001 C CNN
-F 3 "" H 5350 6950 50  0001 C CNN
-	1    5350 6950
-	-1   0    0    1
-$EndComp
-Text Label 5450 6950 3    50   ~ 0
-SDA
-Text Label 5550 6950 3    50   ~ 0
-SCL
-Wire Wire Line
-	5250 6950 5100 6950
 $EndSCHEMATC

Commit message: updating PCB
Parts:
- J4: value Qwiic -> I2C 5v
- U1: value MCP1700-3302E_TO92 -> MCP1700
- U3: footprint ESP8266:ESP-12E_SMD -> RF_Module:ESP-12E; symbol pm_25-rescue:ESP-12F-ESP8266 -> RF_Module:ESP-12F
- U4: value Plantower-PM2.5 -> PM2.5
Connections:
- net +3V3: no longer J4.2 (Pin_2)
- net +5V: now also J4.2 (Pin_2)
- net FLASH: now also U3.18 (GPIO0); no longer U3.12 (GPIO0)
- net GND: now also U3.15 (GND); no longer U3.9 (GND)
- net SCL: now also U3.20 (GPIO5); no longer U3.14 (GPIO5)
- net SDA: now also U3.19 (GPIO4); no longer U3.13 (GPIO4)
- net at R2.1, U4.5 (RX): now also U3.16 (GPIO15); no longer U3.10 (GPIO15)
- net at U2.6 (UTx): now also U3.21 (GPIO3/RXD); no longer U3.15 (RXD)
- net at U2.5 (URx): now also U3.22 (GPIO1/TXD); no longer U3.16 (TXD)
Changed lines of the file:
@@
 P 7250 2750
 F 0 "U4" H 7225 3331 50  0000 C CNN
-F 1 "Plantower-PM2.5" H 7225 3240 50  0000 C CNN
+F 1 "PM2.5" H 7225 3240 50  0000 C CNN
 F 2 "Connector_Molex:Molex_PicoBlade_53261-0871_1x08-1MP_P1.25mm_Horizontal" H 7250 2750 50  0001 C CNN
 F 3 "" H 7250 2750 50  0001 C CNN
@@
 	7250 3100 7250 3150
 $Comp
-L pm_25-rescue:ESP-12F-ESP8266 U3
+L RF_Module:ESP-12F U3
 U 1 1 600365AB
 P 8950 4200
 F 0 "U3" H 8950 4965 50  0000 C CNN
 F 1 "ESP-12F" H 8950 4874 50  0000 C CNN
-F 2 "ESP8266:ESP-12E_SMD" H 8950 4200 50  0001 C CNN
+F 2 "RF_Module:ESP-12E" H 8950 4200 50  0001 C CNN
 F 3 "" H 8950 4200 50  0001 C CNN
 	1    8950 4200
@@
 Wire Wire Line
 	6900 5850 10000 5850
-Wire Wire Line
-	10000 5850 10000 3900
-Wire Wire Line
-	10000 3900 9850 3900
-Text Label 8050 3900 2    50   ~ 0
+Text Label 8350 3600 2    50   ~ 0
 RST
 Text Label 6250 4400 0    50   ~ 0
@@
 Text Label 6250 4300 0    50   ~ 0
 FLASH
-Text Label 9850 4300 0    50   ~ 0
+Text Label 9550 3600 0    50   ~ 0
 FLASH
 $Comp
 L power:+3.3V #PWR0101
 U 1 1 6004A0C6
-P 7650 3950
-F 0 "#PWR0101" H 7650 3800 50  0001 C CNN
-F 1 "+3.3V" H 7665 4123 50  0000 C CNN
-F 2 "" H 7650 3950 50  0001 C CNN
-F 3 "" H 7650 3950 50  0001 C CNN
-	1    7650 3950
-	1    0    0    -1
-$EndComp
-Wire Wire Line
-	8050 4100 7650 4100
-Wire Wire Line
-	7650 4100 7650 3950
-Wire Wire Line
-	8050 4600 7650 4600
-Wire Wire Line
-	7650 4600 7650 4100
-Connection ~ 7650 4100
+P 8950 3400
+F 0 "#PWR0101" H 8950 3250 50  0001 C CNN
+F 1 "+3.3V" H 8965 3573 50  0000 C CNN
+F 2 "" H 8950 3400 50  0001 C CNN
+F 3 "" H 8950 3400 50  0001 C CNN
+	1    8950 3400
+	1    0    0    -1
+$EndComp
 $Comp
 L power:GND #PWR0102
 U 1 1 6004C47E
-P 9850 4750
-F 0 "#PWR0102" H 9850 4500 50  0001 C CNN
-F 1 "GND" H 9855 4577 50  0000 C CNN
-F 2 "" H 9850 4750 50  0001 C CNN
-F 3 "" H 9850 4750 50  0001 C CNN
-	1    9850 4750
-	1    0    0    -1
-$EndComp
-Wire Wire Line
-	9850 4600 9850 4750
+P 8950 4900
+F 0 "#PWR0102" H 8950 4650 50  0001 C CNN
+F 1 "GND" H 8955 4727 50  0000 C CNN
+F 2 "" H 8950 4900 50  0001 C CNN
+F 3 "" H 8950 4900 50  0001 C CNN
+	1    8950 4900
+	1    0    0    -1
+$EndComp
 Text Label 5450 4100 2    50   ~ 0
 D+
@@
 	5850 5100 5850 4800
 Wire Wire Line
-	8050 4500 7850 4500
-Wire Wire Line
-	7850 4500 7850 2900
-Wire Wire Line
-	7850 2900 7550 2900
-Wire Wire Line
-	9850 4500 10450 4500
-Wire Wire Line
 	10450 4500 10450 2600
 Wire Wire Line
@@
 P 4400 2750
 F 0 "U1" H 4400 2508 50  0000 C CNN
-F 1 "MCP1700-3302E_TO92" H 4400 2599 50  0000 C CNN
+F 1 "MCP1700" H 4400 2599 50  0000 C CNN
 F 2 "Package_TO_SOT_THT:TO-92_Inline" H 4400 2550 50  0001 C CIN
 F 3 "http://ww1.microchip.com/downloads/en/DeviceDoc/20001826D.pdf" H 4400 2750 50  0001 C CNN
@@
 Text Label 5500 6300 3    50   ~ 0
 SCL
-Text Label 9850 4200 0    50   ~ 0
+Text Label 9550 4000 0    50   ~ 0
 SDA
-Text Label 9850 4100 0    50   ~ 0
+Text Label 9550 4100 0    50   ~ 0
 SCL
 $Comp
@@
 NoConn ~ 6900 2550
 NoConn ~ 6900 2650
-NoConn ~ 8050 4000
-NoConn ~ 8700 5100
-NoConn ~ 8800 5100
-NoConn ~ 8900 5100
-NoConn ~ 9000 5100
-NoConn ~ 9100 5100
-NoConn ~ 9200 5100
-NoConn ~ 9850 4400
+NoConn ~ 8350 4000
+NoConn ~ 8350 4300
+NoConn ~ 8350 4400
+NoConn ~ 8350 4500
+NoConn ~ 8350 4600
+NoConn ~ 8350 4700
+NoConn ~ 9550 4600
+NoConn ~ 9550 3800
 $Comp
 L Connector:USB_C_Receptacle_USB2.0 J1
@@
 Wire Wire Line
 	5200 6300 5050 6300
-NoConn ~ 8050 4200
-Wire Wire Line
-	8050 4300 6750 4300
-Wire Wire Line
-	6750 4300 6750 4500
-Wire Wire Line
-	6750 4500 6250 4500
-Wire Wire Line
-	8050 4400 6800 4400
-Wire Wire Line
-	6800 4400 6800 4600
-Wire Wire Line
-	6800 4600 6250 4600
+NoConn ~ 8350 4200
 $Comp
 L power:GND #PWR0120
@@
 $EndComp
 $Comp
-L power:+3.3V #PWR0121
-U 1 1 600F9C9F
+L Connector_Generic:Conn_01x04 J4
+U 1 1 600F9C93
+P 5350 6750
+F 0 "J4" V 5314 6462 50  0000 R CNN
+F 1 "I2C 5v" V 5223 6462 50  0000 R CNN
+F 2 "Connector_JST:JST_SH_BM04B-SRSS-TB_1x04-1MP_P1.00mm_Vertical" H 5350 6750 50  0001 C CNN
+F 3 "~" H 5350 6750 50  0001 C CNN
+	1    5350 6750
+	0    -1   -1   0
+$EndComp
+$Comp
+L power:+5V #PWR0121
+U 1 1 602F3278
 P 5350 6950
 F 0 "#PWR0121" H 5350 6800 50  0001 C CNN
-F 1 "+3.3V" H 5365 7123 50  0000 C CNN
+F 1 "+5V" H 5365 7123 50  0000 C CNN
 F 2 "" H 5350 6950 50  0001 C CNN
 F 3 "" H 5350 6950 50  0001 C CNN
@@
 	-1   0    0    1
 $EndComp
-$Comp
-L Connector_Generic:Conn_01x04 J4
-U 1 1 600F9C93
-P 5350 6750
-F 0 "J4" V 5314 6462 50  0000 R CNN
-F 1 "Qwiic" V 5223 6462 50  0000 R CNN
-F 2 "Connector_JST:JST_SH_BM04B-SRSS-TB_1x04-1MP_P1.00mm_Vertical" H 5350 6750 50  0001 C CNN
-F 3 "~" H 5350 6750 50  0001 C CNN
-	1    5350 6750
-	0    -1   -1   0
-$EndComp
+Wire Wire Line
+	10000 3700 9550 3700
+Wire Wire Line
+	10000 3700 10000 5850
+Wire Wire Line
+	9850 4000 9850 3900
+Wire Wire Line
+	9850 3900 9550 3900
+Wire Wire Line
+	9550 4200 9750 4200
+Wire Wire Line
+	9750 4200 9750 5250
+Wire Wire Line
+	9750 5250 6500 5250
+Wire Wire Line
+	6500 5250 6500 4600
+Wire Wire Line
+	6500 4600 6250 4600
+Wire Wire Line
+	9550 4300 10250 4300
+Wire Wire Line
+	10250 4300 10250 2900
+Wire Wire Line
+	7550 2900 10250 2900
+Wire Wire Line
+	9550 4400 9700 4400
+Wire Wire Line
+	9700 4400 9700 5000
+Wire Wire Line
+	9700 5000 6650 5000
+Wire Wire Line
+	6650 5000 6650 4500
+Wire Wire Line
+	6650 4500 6250 4500
+Wire Wire Line
+	9550 4500 10450 4500
+Wire Wire Line
+	8350 3800 7850 3800
+Wire Wire Line
+	7850 3800 7850 3400
+Wire Wire Line
+	7850 3400 8950 3400
+Connection ~ 8950 3400
 $EndSCHEMATC

Commit message: making it look better
Parts:
- J3: value Qwiic -> I2C 3.3v
Changed lines of the file:
@@
 P 5300 6100
 F 0 "J3" V 5264 5812 50  0000 R CNN
-F 1 "Qwiic" V 5173 5812 50  0000 R CNN
+F 1 "I2C 3.3v" V 5173 5812 50  0000 R CNN
 F 2 "Connector_JST:JST_SH_BM04B-SRSS-TB_1x04-1MP_P1.00mm_Vertical" H 5300 6100 50  0001 C CNN
 F 3 "~" H 5300 6100 50  0001 C CNN

Commit message: update pcb with pulldown resistors for USB-C
Parts:
- added R3, R4: 5.1k, Resistor_THT:R_Axial_DIN0207_L6.3mm_D2.5mm_P7.62mm_Horizontal, symbol Device:R
Connections:
- net GND: now also R3.2, R4.2
- net CC1: now reaches J1.A5 (CC1)
- net CC1: now also R3.1
- net CC2: now reaches J1.B5 (CC2)
- net CC2: now also R4.1
- no-connect marks 17 -> 15
Changed lines of the file:
@@
 Sheet 1 1
 Title "PM-2.5 / Temp Wifi Sensor"
-Date "2021-01-16"
+Date "2021-03-09"
 Rev "v04"
 Comp ""
@@
 	1    0    0    -1
 $EndComp
-NoConn ~ 3350 2450
-NoConn ~ 3350 2550
 NoConn ~ 3350 3350
 NoConn ~ 3350 3450
@@
 	7850 3400 8950 3400
 Connection ~ 8950 3400
+$Comp
+L Device:R R3
+U 1 1 60483EC3
+P 2050 5000
+F 0 "R3" H 2120 5046 50  0000 L CNN
+F 1 "5.1k" H 2120 4955 50  0000 L CNN
+F 2 "Resistor_THT:R_Axial_DIN0207_L6.3mm_D2.5mm_P7.62mm_Horizontal" V 1980 5000 50  0001 C CNN
+F 3 "~" H 2050 5000 50  0001 C CNN
+	1    2050 5000
+	1    0    0    -1
+$EndComp
+$Comp
+L Device:R R4
+U 1 1 60484D3B
+P 2450 5000
+F 0 "R4" H 2520 5046 50  0000 L CNN
+F 1 "5.1k" H 2520 4955 50  0000 L CNN
+F 2 "Resistor_THT:R_Axial_DIN0207_L6.3mm_D2.5mm_P7.62mm_Horizontal" V 2380 5000 50  0001 C CNN
+F 3 "~" H 2450 5000 50  0001 C CNN
+	1    2450 5000
+	1    0    0    -1
+$EndComp
+$Comp
+L power:GND #PWR0122
+U 1 1 604854A3
+P 2450 5150
+F 0 "#PWR0122" H 2450 4900 50  0001 C CNN
+F 1 "GND" H 2455 4977 50  0000 C CNN
+F 2 "" H 2450 5150 50  0001 C CNN
+F 3 "" H 2450 5150 50  0001 C CNN
+	1    2450 5150
+	1    0    0    -1
+$EndComp
+$Comp
+L power:GND #PWR0123
+U 1 1 604859C1
+P 2050 5150
+F 0 "#PWR0123" H 2050 4900 50  0001 C CNN
+F 1 "GND" H 2055 4977 50  0000 C CNN
+F 2 "" H 2050 5150 50  0001 C CNN
+F 3 "" H 2050 5150 50  0001 C CNN
+	1    2050 5150
+	1    0    0    -1
+$EndComp
+Text Label 3350 2450 0    50   ~ 0
+CC1
+Text Label 3350 2550 0    50   ~ 0
+CC2
+Text Label 2050 4850 0    50   ~ 0
+CC1
+Text Label 2450 4850 0    50   ~ 0
+CC2
 $EndSCHEMATC
